Commit message: update to work

File: src/so_arm101_description/urdf/so_arm_101_simplified_best.urdf (robot description, URDF)
Before this commit: robot so100, 10 links, 9 joints
Joints:
- joint joint_1: limit lower=-1.91986 upper=1.91986 effort=10 velocity=10 -> lower=-1.57 upper=1.57 effort=10 velocity=10
- joint joint_2: limit lower=-1.74533 upper=1.74533 effort=10 velocity=10 -> lower=-1.57 upper=1.57 effort=10 velocity=10
- joint joint_3: limit lower=-1.74533 upper=1.5708 effort=10 velocity=10 -> lower=-1.5359 upper=1.5359 effort=10 velocity=10
- joint joint_4: limit lower=-1.65806 upper=1.65806 effort=10 velocity=10 -> lower=-1.5359 upper=1.5359 effort=10 velocity=10
- joint joint_5: limit lower=-2.74385 upper=2.84121 effort=10 velocity=10 -> lower=-2.6180 upper=2.6180 effort=10 velocity=10
- joint joint_6: limit lower=-0.174533 upper=1.74533 effort=10 velocity=10 -> lower=0.00 upper=1.5708 effort=10 velocity=10

File: src/so_arm101_moveit_config/config/so100.ros2_control.xacro (robot description, xacro)
@@ -5,48 +5,35 @@
         <ros2_control name="${name}" type="system">
             <hardware>
-                <!-- By default, set up controllers for simulation. This won't work on real hardware -->
-                <plugin>mock_components/GenericSystem</plugin>
+                <plugin>so101_hardware/SO101HardwareInterface</plugin>
+                <param name="device">/dev/ttyUSB0</param>
             </hardware>
             <joint name="joint_1">
-                <command_interface name="position"/>
-                <state_interface name="position">
-                  <param name="initial_value">0.0</param>
-                </state_interface>
-                <state_interface name="velocity"/>
+                <param name="id">1</param> <command_interface name="position"/>
+                <state_interface name="position"/>
             </joint>
             <joint name="joint_2">
+                <param name="id">2</param>
                 <command_interface name="position"/>
-                <state_interface name="position">
-                  <param name="initial_value">0.0</param>
-                </state_interface>
-                <state_interface name="velocity"/>
+                <state_interface name="position"/>
             </joint>
             <joint name="joint_3">
+                <param name="id">3</param>
                 <command_interface name="position"/>
-                <state_interface name="position">
-                  <param name="initial_value">0.0</param>
-                </state_interface>
-                <state_interface name="velocity"/>
+                <state_interface name="position"/>
             </joint>
             <joint name="joint_4">
+                <param name="id">4</param>
                 <command_interface name="position"/>
-                <state_interface name="position">
-                  <param name="initial_value">0.0</param>
-                </state_interface>
-                <state_interface name="velocity"/>
+                <state_interface name="position"/>
             </joint>
             <joint name="joint_5">
+                <param name="id">5</param>
                 <command_interface name="position"/>
-                <state_interface name="position">
-                  <param name="initial_value">0.0</param>
-                </state_interface>
-                <state_interface name="velocity"/>
+                <state_interface name="position"/>
             </joint>
             <joint name="joint_6">
+                <param name="id">6</param>
                 <command_interface name="position"/>
-                <state_interface name="position">
-                  <param name="initial_value">0.0</param>
-                </state_interface>
-                <state_interface name="velocity"/>
+                <state_interface name="position"/>
             </joint>
         </ros2_control>
